File: schematic/Micro-USB-UART.kicad_pcb (KiCad board)
At the start: 2 copper layers, 25.4 x 19 mm, 14 parts, among them IC1 CP2102N-A01-GQFN28R, J1 Conn_01x09, J2 Conn_01x09, U1 DizzyBITLogo

Commit message: Updated
Parts:
- moved J2 0.14 mm to (75.4, 121.8)
Routing:
- net GND: track 7.39 -> 9.76 mm
- net EXT_5V: track 17.5 -> 18.9 mm
- net VBUS: track 20.5 -> 21.9 mm
Other:
- board size 25.4 x 19 mm -> 25.4 x 15.2 mm
- net class Default: clearance 0.2 -> 0.1
- rule trace_clearance: 0.2 -> 0.1
Changed lines of the file:
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@@
     (thickness 1.6)
     (drawings 5)
-    (tracks 98)
+    (tracks 100)
     (zones 0)
     (modules 14)
@@
     (35 F.Paste user)
     (36 B.SilkS user)
-    (37 F.SilkS user hide)
+    (37 F.SilkS user)
     (38 B.Mask user)
     (39 F.Mask user)
@@
   )
   (setup
-    (last_trace_width 0.508)
+    (last_trace_width 1)
     (user_trace_width 0.25)
     (user_trace_width 0.508)
     (user_trace_width 1)
     (user_trace_width 2)
-    (trace_clearance 0.2)
+    (trace_clearance 0.1)
     (zone_clearance 0.254)
     (zone_45_only no)
@@
   (net 12 DTR)
   (net_class Default "This is the default net class."
-    (clearance 0.2)
+    (clearance 0.1)
     (trace_width 0.25)
     (via_dia 0.8)
@@
     (descr "Through hole straight socket strip, 1x09, 2.54mm pitch, single row (from Kicad 4.0.7), script generated")
     (tags "Through hole socket strip THT 1x09 2.54mm single row")
-    (fp_text reference J1 (at 0 -2.77 270) (layer F.SilkS)
+    (fp_text reference J1 (at -0.1143 -1.9304 270) (layer F.SilkS)
       (effects (font (size 1 1) (thickness 0.15)))
     )
@@
   )
   (module Connector_PinSocket_2.54mm:PinSocket_1x09_P2.54mm_Vertical (layer F.Cu)
-    (at 75.438 121.6152 90)
+    (at 75.438 121.7549 90)
     (descr "Through hole straight socket strip, 1x09, 2.54mm pitch, single row (from Kicad 4.0.7), script generated")
     (tags "Through hole socket strip THT 1x09 2.54mm single row")
@@
     (effects (font (size 1 1) (thickness 0.2)) (justify mirror))
   )
-  (gr_line (start 98.298 123.7488) (end 98.298 104.7496) (layer Edge.Cuts) (width 0.15))
-  (gr_line (start 72.898 123.7488) (end 72.898 104.7496) (layer Edge.Cuts) (width 0.15))
-  (gr_line (start 98.298 123.7488) (end 72.898 123.7488) (layer Edge.Cuts) (width 0.15))
-  (gr_line (start 72.898 104.7496) (end 98.298 104.7496) (layer Edge.Cuts) (width 0.15))
+  (gr_line (start 98.298 121.7549) (end 98.298 106.5276) (layer Edge.Cuts) (width 0.15))
+  (gr_line (start 72.898 121.7549) (end 72.898 106.5276) (layer Edge.Cuts) (width 0.15))
+  (gr_line (start 98.298 121.7549) (end 72.898 121.7549) (layer Edge.Cuts) (width 0.15))
+  (gr_line (start 72.898 106.5276) (end 98.298 106.5276) (layer Edge.Cuts) (width 0.15))
   (via (at 87.376 114.8588) (size 0.8) (drill 0.4) (layers F.Cu B.Cu) (net 1))
   (via (at 91.5416 117.8052) (size 0.8) (drill 0.4) (layers F.Cu B.Cu) (net 1))
@@
   (segment (start 90.9908 112.9872) (end 91.4908 113.4872) (width 0.25) (layer F.Cu) (net 1))
   (segment (start 89.1408 112.9872) (end 90.9908 112.9872) (width 0.25) (layer F.Cu) (net 1))
-  (segment (start 83.5025 110.0455) (end 81.4705 108.0135) (width 1) (layer F.Cu) (net 1))
   (segment (start 83.5025 111.291) (end 83.5025 111.252) (width 1) (layer F.Cu) (net 1))
-  (segment (start 83.5025 111.252) (end 83.5025 110.0455) (width 1) (layer F.Cu) (net 1))
-  (via (at 83.5025 111.252) (size 0.8) (drill 0.4) (layers F.Cu B.Cu) (net 1))
   (via (at 92.5576 112.4712) (size 0.8) (drill 0.4) (layers F.Cu B.Cu) (net 1))
   (via (at 92.5068 114.5032) (size 0.8) (drill 0.4) (layers F.Cu B.Cu) (net 1))
   (via (at 90.4748 114.4524) (size 0.8) (drill 0.4) (layers F.Cu B.Cu) (net 1))
-  (segment (start 81.4705 108.0135) (end 81.4705 107.30261) (width 1) (layer F.Cu) (net 1))
+  (segment (start 83.5025 109.5121) (end 83.5025 111.252) (width 1) (layer F.Cu) (net 1))
+  (segment (start 80.518 106.5276) (end 83.5025 109.5121) (width 1) (layer F.Cu) (net 1))
+  (via (at 83.5025 111.252) (size 0.8) (drill 0.4) (layers F.Cu B.Cu) (net 1))
+  (segment (start 83.5025 111.252) (end 83.5025 110.0455) (width 1) (layer F.Cu) (net 1))
   (segment (start 87.6944 116.4336) (end 89.115799 115.012201) (width 1) (layer F.Cu) (net 2))
   (segment (start 85.852 116.4336) (end 87.6944 116.4336) (width 1) (layer F.Cu) (net 2))
   (segment (start 89.1408 114.4872) (end 89.1408 114.9872) (width 0.25) (layer F.Cu) (net 2))
-  (segment (start 85.598 121.6152) (end 83.058 121.6152) (width 2) (layer F.Cu) (net 2))
   (segment (start 85.852 121.3612) (end 85.598 121.6152) (width 1) (layer F.Cu) (net 2))
   (segment (start 85.852 116.4336) (end 85.852 120.0404) (width 1) (layer F.Cu) (net 2))
@@
   (segment (start 92.17409 120.24621) (end 86.96699 120.24621) (width 0.508) (layer F.Cu) (net 2))
   (segment (start 93.0656 119.3547) (end 92.17409 120.24621) (width 0.508) (layer F.Cu) (net 2))
+  (segment (start 83.058 121.7549) (end 85.598 121.7549) (width 2) (layer F.Cu) (net 2))
   (via (at 89.1032 119.38) (size 0.8) (drill 0.4) (layers F.Cu B.Cu) (net 3))
   (via (at 81.4324 110.6424) (size 0.8) (drill 0.4) (layers F.Cu B.Cu) (net 3))
@@
   (segment (start 84.582 119.38) (end 81.032401 115.830401) (width 2) (layer B.Cu) (net 3))
   (segment (start 89.1032 119.38) (end 84.582 119.38) (width 2) (layer B.Cu) (net 3))
+  (segment (start 88.138 121.6152) (end 88.138 120.3452) (width 2) (layer B.Cu) (net 3))
   (segment (start 88.138 120.3452) (end 89.1032 119.38) (width 2) (layer B.Cu) (net 3))
-  (segment (start 88.138 121.6152) (end 88.138 120.3452) (width 2) (layer B.Cu) (net 3))
+  (segment (start 88.138 121.7549) (end 88.138 120.3452) (width 2) (layer B.Cu) (net 3))
   (segment (start 81.4125 112.991) (end 81.407 112.9855) (width 1) (layer F.Cu) (net 4))
   (segment (start 83.5025 112.991) (end 83.4644 112.9792) (width 1) (layer F.Cu) (net 4))
@@
   (segment (start 81.3371 112.9855) (end 80.8736 112.522) (width 1) (layer F.Cu) (net 4))
   (segment (start 80.8736 112.522) (end 78.3336 112.522) (width 1) (layer F.Cu) (net 4))
-  (segment (start 90.678 120.413119) (end 90.8812 120.209919) (width 1) (layer B.Cu) (net 4))
   (segment (start 90.678 121.6152) (end 90.678 120.413119) (width 1) (layer B.Cu) (net 4))
   (segment (start 90.8812 118.753822) (end 88.8492 116.721822) (width 1) (layer B.Cu) (net 4))
   (segment (start 90.8812 120.209919) (end 90.8812 118.753822) (width 1) (layer B.Cu) (net 4))
+  (segment (start 90.678 120.413119) (end 90.8812 120.209919) (width 1) (layer B.Cu) (net 4))
+  (segment (start 90.678 121.7549) (end 90.678 120.413119) (width 1) (layer B.Cu) (net 4))
   (segment (start 81.39685 114.90325) (end 81.534 114.7661) (width 0.25) (layer F.Cu) (net 5))
   (segment (start 81.534 114.7661) (end 81.634 114.7661) (width 0.25) (layer F.Cu) (net 5))
